Commit message: added support for gazebo

File: src/robot_urdf/urdf/robot.urdf.xacro (robot description, xacro)
@@ -1,16 +1,4 @@
 <?xml version="1.0"?>
 <robot xmlns:xacro="http://www.ros.org/wiki/xacro" name="robot">
-  <material name="blue">
-    <color rgba="0 0 0.8 .5"/>
-  </material>
-  <material name="black">
-    <color rgba="0 0 0 0.5"/>
-  </material>
-  <material name="white">
-    <color rgba="1 1 1 .5"/>
-  </material>
-  <material name="green">
-    <color rgba="0 1 0 0.5"/>
-  </material>
   <xacro:property name="baseLength" value="0.8255" />
   <xacro:property name="baseWidth" value="0.6985" />
@@ -24,4 +12,8 @@
   <xacro:property name="camWidth" value="0.1016" />
   <xacro:property name="camRadius" value="0.0127" />
+  <!-- Import all Gazebo-customization elements, including Gazebo colors -->
+  <xacro:include filename="$(find robot_urdf)/urdf/robot.gazebo" />
+  <!-- Import Rviz colors -->
+  <xacro:include filename="$(find robot_urdf)/urdf/materials.xacro" />
   <link name="base_link">
     <visual>
@@ -142,78 +134,29 @@
   </joint>
   <!-- Sensors -->
-  <link name="t265_pose_frame">
+  <!-- Hokuyo Laser -->
+  <link name="hokuyo_link">
+    <collision>
+      <origin xyz="0 0 0" rpy="0 0 0"/>
+      <geometry>
+	<box size="0.1 0.1 0.1"/>
+      </geometry>
+    </collision>
     <visual>
+      <origin xyz="0 0 0" rpy="0 0 0"/>
       <geometry>
-        <cylinder length="${camWidth}" radius="${camRadius}"/>
+        <mesh filename="package://robot_urdf/meshes/hokuyo.dae"/>
       </geometry>
-      <origin rpy="0 1.57075 1.57075" xyz="0 0 0"/>
-      <material name="white"/>
     </visual>
-    <collision>
-      <geometry>
-        <cylinder length="${camWidth}" radius="${camRadius}"/>
-      </geometry>
-      <origin rpy="0 1.57075 1.57075" xyz="0 0 0"/>
-    </collision>
     <inertial>
-      <mass value="${camMass}"/>
-      <inertia ixx="0.4" ixy="0.0" ixz="0.0" iyy="0.4" iyz="0.0" izz="0.2"/>
+      <mass value="1e-5" />
+      <origin xyz="0 0 0" rpy="0 0 0"/>
+      <inertia ixx="1e-6" ixy="0" ixz="0" iyy="1e-6" iyz="0" izz="1e-6" />
     </inertial>
   </link>
-  <joint name="base_to_t265_pose_frame" type="fixed">
+  <joint name="hokuyo_joint" type="fixed">
+    <axis xyz="0 1 0" />
+    <origin xyz="0 0 0.4" rpy="0 0 0"/>
     <parent link="base_link"/>
-    <child link="t265_pose_frame"/>
-    <axis xyz="0 1 0"/>
-    <origin xyz="0.2159 0 .2"/>
-  </joint>
-  <link name="d435_link">
-    <visual>
-      <geometry>
-        <cylinder length="${camWidth}" radius="${camRadius}"/>
-      </geometry>
-      <origin rpy="0 1.57075 1.57075" xyz="0 0 0"/>
-      <material name="white"/>
-    </visual>
-    <collision>
-      <geometry>
-        <cylinder length="${camWidth}" radius="${camRadius}"/>
-      </geometry>
-      <origin rpy="0 1.57075 1.57075" xyz="0 0 0"/>
-    </collision>
-    <inertial>
-      <mass value="${camMass}"/>
-      <inertia ixx="0.4" ixy="0.0" ixz="0.0" iyy="0.4" iyz="0.0" izz="0.2"/>
-    </inertial>
-  </link>
-  <joint name="base_to_d435_link" type="fixed">
-    <parent link="base_link"/>
-    <child link="d435_link"/>
-    <axis xyz="0 1 0"/>
-    <origin xyz="0.2159 0 0.2508"/>
-  </joint>
-  <link name="laser">
-    <visual>
-      <geometry>
-        <cylinder length="${camWidth}" radius="${camRadius}"/>
-      </geometry>
-      <origin rpy="0 1.57075 1.57075" xyz="0 0 0"/>
-      <material name="white"/>
-    </visual>
-    <collision>
-      <geometry>
-        <cylinder length="${camWidth}" radius="${camRadius}"/>
-      </geometry>
-      <origin rpy="0 1.57075 1.57075" xyz="0 0 0"/>
-    </collision>
-    <inertial>
-      <mass value="${camMass}"/>
-      <inertia ixx="0.4" ixy="0.0" ixz="0.0" iyy="0.4" iyz="0.0" izz="0.2"/>
-    </inertial>
-  </link>
-  <joint name="base_to_laser" type="fixed">
-    <parent link="base_link"/>
-    <child link="laser"/>
-    <axis xyz="0 1 0"/>
-    <origin xyz="0.2159 0 0.2508" rpy="0 0 3.1415"/>
+    <child link="hokuyo_link"/>
   </joint>
 </robot>

Commit message: added lidar

File: src/robot_urdf/urdf/robot.urdf.xacro (robot description, xacro)
@@ -135,4 +135,10 @@
   <!-- Sensors -->
   <!-- Hokuyo Laser -->
+  <joint name="hokuyo_joint" type="fixed">
+    <axis xyz="0 1 0" />
+    <origin xyz="0 0 0.4" rpy="0 0 0"/>
+    <parent link="base_link"/>
+    <child link="hokuyo_link"/>
+  </joint>
   <link name="hokuyo_link">
     <collision>
@@ -154,9 +160,3 @@
     </inertial>
   </link>
-  <joint name="hokuyo_joint" type="fixed">
-    <axis xyz="0 1 0" />
-    <origin xyz="0 0 0.4" rpy="0 0 0"/>
-    <parent link="base_link"/>
-    <child link="hokuyo_link"/>
-  </joint>
 </robot>

Commit message: added gazebo world

File: src/robot_urdf/urdf/robot.urdf.xacro (robot description, xacro)
@@ -137,5 +137,5 @@
   <joint name="hokuyo_joint" type="fixed">
     <axis xyz="0 1 0" />
-    <origin xyz="0 0 0.4" rpy="0 0 0"/>
+    <origin xyz="0.41275 0 0.35" rpy="0 0 0"/>
     <parent link="base_link"/>
     <child link="hokuyo_link"/>

Commit message: added kinect

File: src/robot_urdf/urdf/robot.urdf.xacro (robot description, xacro)
@@ -145,5 +145,5 @@
       <origin xyz="0 0 0" rpy="0 0 0"/>
       <geometry>
-	<box size="0.1 0.1 0.1"/>
+	      <box size="0.1 0.1 0.1"/>
       </geometry>
     </collision>
@@ -160,3 +160,29 @@
     </inertial>
   </link>
+  <!-- Kinect -->
+  <joint name="kinect_joint" type="fixed">
+    <axis xyz="0 0 0" />
+    <origin xyz="0.41275 0 0.225" rpy="0 0 0"/>
+    <parent link="base_link"/>
+    <child link="kinect_link"/>
+  </joint>
+  <link name="kinect_link">
+    <collision>
+      <origin xyz="0 0 0" rpy="0 0 0"/>
+      <geometry>
+	      <box size="0.02 0.07 0.02"/>
+      </geometry>
+    </collision>
+    <visual>
+      <origin xyz="0 0 0" rpy="0 0 0"/>
+      <geometry>
+        <box size="0.02 0.07 0.02"/>
+      </geometry>
+    </visual>
+    <inertial>
+      <mass value="1e-5" />
+      <origin xyz="0 0 0" rpy="0 0 0"/>
+      <inertia ixx="1e-6" ixy="0" ixz="0" iyy="1e-6" iyz="0" izz="1e-6" />
+    </inertial>
+  </link>
 </robot>

Commit message: added new world

File: src/robot_urdf/urdf/robot.urdf.xacro (robot description, xacro)
@@ -135,11 +135,11 @@
   <!-- Sensors -->
   <!-- Hokuyo Laser -->
-  <joint name="hokuyo_joint" type="fixed">
+  <joint name="laser_joint" type="fixed">
     <axis xyz="0 1 0" />
     <origin xyz="0.41275 0 0.35" rpy="0 0 0"/>
     <parent link="base_link"/>
-    <child link="hokuyo_link"/>
+    <child link="laser"/>
   </joint>
-  <link name="hokuyo_link">
+  <link name="laser">
     <collision>
       <origin xyz="0 0 0" rpy="0 0 0"/>
@@ -160,12 +160,12 @@
     </inertial>
   </link>
-  <!-- Kinect -->
-  <joint name="kinect_joint" type="fixed">
+  <!-- Kinect
+  <joint name="d435_joint" type="fixed">
     <axis xyz="0 0 0" />
     <origin xyz="0.41275 0 0.225" rpy="0 0 0"/>
     <parent link="base_link"/>
-    <child link="kinect_link"/>
+    <child link="d435_link"/>
   </joint>
-  <link name="kinect_link">
+  <link name="d435_link">
     <collision>
       <origin xyz="0 0 0" rpy="0 0 0"/>
@@ -186,3 +186,4 @@
     </inertial>
   </link>
+  -->
 </robot>
